Commit message: updated our g1 module to work with ros2

File: robots/g1_description/g1_29dof_rev_1_0_with_inspire_hand_FTP.urdf (robot description, URDF)
Before this commit: robot g1_29dof_rev_1_0_with_inspire_hand_FTP, 97 links, 96 joints
Links:
- link head_link: geometry collision mesh filename=package://unitree_ros2/description/g1/meshes/head_link.STL; visual mesh filename=package://unitree_ros2/description/g1/meshes/head_link.STL
- link left_ankle_pitch_link: geometry collision mesh filename=package://unitree_ros2/description/g1/meshes/left_ankle_pit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; visual mesh filename=package://unitree_ros2/description/g1/meshes/left_ankle_pit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
- link left_ankle_roll_link: geometry collision sphere radius=0.005; collision sphere radius=0.005
- link left_base_link: geometry collision mesh filename=package://unitree_ros2/description/g1/meshes/left_base_link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; visual mesh filename=package://unitree_ros2/description/g1/meshes/left_base_link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
- link left_elbow_link: geometry collision mesh filename=package://unitree_ros2/description/g1/meshes/left_elbow_lin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; visual mesh filename=package://unitree_ros2/description/g1/meshes/left_elbow_lin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
- link left_hip_pitch_link: geometry collision mesh filename=package://unitree_ros2/description/g1/meshes/left_hip_pitch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; visual mesh filename=package://unitree_ros2/description/g1/meshes/left_hip_pitch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
- link left_hip_roll_link: geometry collision mesh filename=package://unitree_ros2/description/g1/meshes/left_hip_roll_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; visual mesh filename=package://unitree_ros2/description/g1/meshes/left_hip_roll_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
- link left_hip_yaw_link: geometry collision mesh filename=package://unitree_ros2/description/g1/meshes/left_hip_yaw_l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; visual mesh filename=package://unitree_ros2/description/g1/meshes/left_hip_yaw_l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
- link left_index_1: geometry collision mesh filename=package://unitree_ros2/description/g1/meshes/left_index_1.S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; visual mesh filename=package://unitree_ros2/description/g1/meshes/left_index_1.S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
- link left_index_2: geometry collision mesh filename=package://unitree_ros2/description/g1/meshes/left_index_2.S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; visual mesh filename=package://unitree_ros2/description/g1/meshes/left_index_2.S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
- link left_index_force_sensor_1: geometry collision mesh filename=package://unitree_ros2/description/g1/meshes/left_index_for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; visual mesh filename=package://unitree_ros2/description/g1/meshes/left_index_for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
- link left_index_force_sensor_2: geometry collision mesh filename=package://unitree_ros2/description/g1/meshes/left_index_for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; visual mesh filename=package://unitree_ros2/description/g1/meshes/left_index_for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
- link left_index_force_sensor_3: geometry collision mesh filename=package://unitree_ros2/description/g1/meshes/left_index_for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; visual mesh filename=package://unitree_ros2/description/g1/meshes/left_index_for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
- link left_knee_link: geometry collision mesh filename=package://unitree_ros2/description/g1/meshes/left_knee_link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; visual mesh filename=package://unitree_ros2/description/g1/meshes/left_knee_link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
- link left_little_1: geometry collision mesh filename=package://unitree_ros2/description/g1/meshes/left_little_1.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; visual mesh filename=package://unitree_ros2/description/g1/meshes/left_little_1.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
- link left_little_2: geometry collision mesh filename=package://unitree_ros2/description/g1/meshes/left_little_2.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; visual mesh filename=package://unitree_ros2/description/g1/meshes/left_little_2.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
- link left_little_force_sensor_1: geometry collision mesh filename=package://unitree_ros2/description/g1/meshes/left_little_fo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; visual mesh filename=package://unitree_ros2/description/g1/meshes/left_little_fo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
- link left_little_force_sensor_2: geometry collision mesh filename=package://unitree_ros2/description/g1/meshes/left_little_fo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; visual mesh filename=package://unitree_ros2/description/g1/meshes/left_little_fo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
- link left_little_force_sensor_3: geometry collision mesh filename=package://unitree_ros2/description/g1/meshes/left_little_fo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; visual mesh filename=package://unitree_ros2/description/g1/meshes/left_little_fo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
- link left_middle_1: geometry collision mesh filename=package://unitree_ros2/description/g1/meshes/left_middle_1.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; visual mesh filename=package://unitree_ros2/description/g1/meshes/left_middle_1.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
- link left_middle_2: geometry collision mesh filename=package://unitree_ros2/description/g1/meshes/left_middle_2.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; visual mesh filename=package://unitree_ros2/description/g1/meshes/left_middle_2.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
- link left_middle_force_sensor_1: geometry collision mesh filename=package://unitree_ros2/description/g1/meshes/left_middle_fo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; visual mesh filename=package://unitree_ros2/description/g1/meshes/left_middle_fo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
- link left_middle_force_sensor_2: geometry collision mesh filename=package://unitree_ros2/description/g1/meshes/left_middle_fo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; visual mesh filename=package://unitree_ros2/description/g1/meshes/left_middle_fo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
- link left_middle_force_sensor_3: geometry collision mesh filename=package://unitree_ros2/description/g1/meshes/left_middle_fo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; visual mesh filename=package://unitree_ros2/description/g1/meshes/left_middle_fo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
- link left_palm_force_sensor: geometry collision mesh filename=package://unitree_ros2/description/g1/meshes/left_palm_forc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; visual mesh filename=package://unitree_ros2/description/g1/meshes/left_palm_forc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
- link left_ring_1: geometry collision mesh filename=package://unitree_ros2/description/g1/meshes/left_ring_1.STL; visual mesh filename=package://unitree_ros2/description/g1/meshes/left_ring_1.STL
- link left_ring_2: geometry collision mesh filename=package://unitree_ros2/description/g1/meshes/left_ring_2.STL; visual mesh filename=package://unitree_ros2/description/g1/meshes/left_ring_2.STL
- link left_ring_force_sensor_1: geometry collision mesh filename=package://unitree_ros2/description/g1/meshes/left_ring_forc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; visual mesh filename=package://unitree_ros2/description/g1/meshes/left_ring_forc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
- link left_ring_force_sensor_2: geometry collision mesh filename=package://unitree_ros2/description/g1/meshes/left_ring_forc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; visual mesh filename=package://unitree_ros2/description/g1/meshes/left_ring_forc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
- link left_ring_force_sensor_3: geometry collision mesh filename=package://unitree_ros2/description/g1/meshes/left_ring_forc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; visual mesh filename=package://unitree_ros2/description/g1/meshes/left_ring_forc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
- link left_shoulder_pitch_link: geometry collision cylinder length=0.05 radius=0.03; visual mesh filename=package://unitree_ros2/description/g1/meshes/left_shoulder_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
- link left_shoulder_roll_link: geometry collision cylinder length=0.03 radius=0.03; visual mesh filename=package://unitree_ros2/description/g1/meshes/left_shoulder_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
- link left_shoulder_yaw_link: geometry collision mesh filename=package://unitree_ros2/description/g1/meshes/left_shoulder_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; visual mesh filename=package://unitree_ros2/description/g1/meshes/left_shoulder_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
- link left_thumb_1: geometry collision mesh filename=package://unitree_ros2/description/g1/meshes/left_thumb_1.S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; visual mesh filename=package://unitree_ros2/description/g1/meshes/left_thumb_1.S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
- link left_thumb_2: geometry collision mesh filename=package://unitree_ros2/description/g1/meshes/left_thumb_2.S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; visual mesh filename=package://unitree_ros2/description/g1/meshes/left_thumb_2.S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
- link left_thumb_3: geometry collision mesh filename=package://unitree_ros2/description/g1/meshes/left_thumb_3.S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; visual mesh filename=package://unitree_ros2/description/g1/meshes/left_thumb_3.S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
- link left_thumb_4: geometry collision mesh filename=package://unitree_ros2/description/g1/meshes/left_thumb_4.S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; visual mesh filename=package://unitree_ros2/description/g1/meshes/left_thumb_4.S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
- link left_thumb_force_sensor_1: geometry collision mesh filename=package://unitree_ros2/description/g1/meshes/left_thumb_for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; visual mesh filename=package://unitree_ros2/description/g1/meshes/left_thumb_for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
- link left_thumb_force_sensor_2: geometry collision mesh filename=package://unitree_ros2/description/g1/meshes/left_thumb_for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; visual mesh filename=package://unitree_ros2/description/g1/meshes/left_thumb_for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
- link left_thumb_force_sensor_3: geometry collision mesh filename=package://unitree_ros2/description/g1/meshes/left_thumb_for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; visual mesh filename=package://unitree_ros2/description/g1/meshes/left_thumb_for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
- link left_thumb_force_sensor_4: geometry collision mesh filename=package://unitree_ros2/description/g1/meshes/left_thumb_for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; visual mesh filename=package://unitree_ros2/description/g1/meshes/left_thumb_for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
- link left_wrist_pitch_link: geometry collision mesh filename=package://unitree_ros2/description/g1/meshes/left_wrist_pit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; visual mesh filename=package://unitree_ros2/description/g1/meshes/left_wrist_pit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
- link left_wrist_roll_link: geometry collision mesh filename=package://unitree_ros2/description/g1/meshes/left_wrist_rol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; visual mesh filename=package://unitree_ros2/description/g1/meshes/left_wrist_rol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
- link left_wrist_yaw_link: geometry collision mesh filename=package://unitree_ros2/description/g1/meshes/left_wrist_yaw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; visual mesh filename=package://unitree_ros2/description/g1/meshes/left_wrist_yaw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
- link logo_link: geometry collision mesh filename=package://unitree_ros2/description/g1/meshes/logo_link.STL; visual mesh filename=package://unitree_ros2/description/g1/meshes/logo_link.STL
- link pelvis: geometry visual mesh filename=package://unitree_ros2/description/g1/meshes/pelvis.STL
- link pelvis_contour_link: geometry collision mesh filename=package://unitree_ros2/description/g1/meshes/pelvis_contour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; visual mesh filename=package://unitree_ros2/description/g1/meshes/pelvis_contour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
- link right_ankle_pitch_link: geometry collision mesh filename=package://unitree_ros2/description/g1/meshes/right_ankle_pi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; visual mesh filename=package://unitree_ros2/description/g1/meshes/right_ankle_pi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
- link right_ankle_roll_link: geometry collision sphere radius=0.005; collision sphere radius=0.005
- link right_base_link: geometry collision mesh filename=package://unitree_ros2/description/g1/meshes/right_base_lin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; visual mesh filename=package://unitree_ros2/description/g1/meshes/right_base_lin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
- link right_elbow_link: geometry collision mesh filename=package://unitree_ros2/description/g1/meshes/right_elbow_li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; visual mesh filename=package://unitree_ros2/description/g1/meshes/right_elbow_li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
- link right_hip_pitch_link: geometry collision mesh filename=package://unitree_ros2/description/g1/meshes/right_hip_pitc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; visual mesh filename=package://unitree_ros2/description/g1/meshes/right_hip_pitc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
- link right_hip_roll_link: geometry collision mesh filename=package://unitree_ros2/description/g1/meshes/right_hip_roll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; visual mesh filename=package://unitree_ros2/description/g1/meshes/right_hip_roll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
- link right_hip_yaw_link: geometry collision mesh filename=package://unitree_ros2/description/g1/meshes/right_hip_yaw_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; visual mesh filename=package://unitree_ros2/description/g1/meshes/right_hip_yaw_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
- link right_index_1: geometry collision mesh filename=package://unitree_ros2/description/g1/meshes/right_index_1.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; visual mesh filename=package://unitree_ros2/description/g1/meshes/right_index_1.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
- link right_index_2: geometry collision mesh filename=package://unitree_ros2/description/g1/meshes/right_index_2.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; visual mesh filename=package://unitree_ros2/description/g1/meshes/right_index_2.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
- link right_index_force_sensor_1: geometry collision mesh filename=package://unitree_ros2/description/g1/meshes/right_index_fo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; visual mesh filename=package://unitree_ros2/description/g1/meshes/right_index_fo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
- link right_index_force_sensor_2: geometry collision mesh filename=package://unitree_ros2/description/g1/meshes/right_index_fo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; visual mesh filename=package://unitree_ros2/description/g1/meshes/right_index_fo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
- link right_index_force_sensor_3: geometry collision mesh filename=package://unitree_ros2/description/g1/meshes/right_index_fo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; visual mesh filename=package://unitree_ros2/description/g1/meshes/right_index_fo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
- link right_knee_link: geometry collision mesh filename=package://unitree_ros2/description/g1/meshes/right_knee_lin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; visual mesh filename=package://unitree_ros2/description/g1/meshes/right_knee_lin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
- link right_little_1: geometry collision mesh filename=package://unitree_ros2/description/g1/meshes/right_little_1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; visual mesh filename=package://unitree_ros2/description/g1/meshes/right_little_1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
- link right_little_2: geometry collision mesh filename=package://unitree_ros2/description/g1/meshes/right_little_2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; visual mesh filename=package://unitree_ros2/description/g1/meshes/right_little_2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
- link right_little_force_sensor_1: geometry collision mesh filename=package://unitree_ros2/description/g1/meshes/right_little_f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; visual mesh filename=package://unitree_ros2/description/g1/meshes/right_little_f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
- link right_little_force_sensor_2: geometry collision mesh filename=package://unitree_ros2/description/g1/meshes/right_little_f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; visual mesh filename=package://unitree_ros2/description/g1/meshes/right_little_f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
- link right_little_force_sensor_3: geometry collision mesh filename=package://unitree_ros2/description/g1/meshes/right_little_f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; visual mesh filename=package://unitree_ros2/description/g1/meshes/right_little_f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
- link right_middle_1: geometry collision mesh filename=package://unitree_ros2/description/g1/meshes/right_middle_1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; visual mesh filename=package://unitree_ros2/description/g1/meshes/right_middle_1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
- link right_middle_2: geometry collision mesh filename=package://unitree_ros2/description/g1/meshes/right_middle_2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; visual mesh filename=package://unitree_ros2/description/g1/meshes/right_middle_2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
- link right_middle_force_sensor_1: geometry collision mesh filename=package://unitree_ros2/description/g1/meshes/right_middle_f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; visual mesh filename=package://unitree_ros2/description/g1/meshes/right_middle_f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
- link right_middle_force_sensor_2: geometry collision mesh filename=package://unitree_ros2/description/g1/meshes/right_middle_f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; visual mesh filename=package://unitree_ros2/description/g1/meshes/right_middle_f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
- link right_middle_force_sensor_3: geometry collision mesh filename=package://unitree_ros2/description/g1/meshes/right_middle_f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; visual mesh filename=package://unitree_ros2/description/g1/meshes/right_middle_f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
- link right_palm_force_sensor: geometry collision mesh filename=package://unitree_ros2/description/g1/meshes/right_palm_for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; visual mesh filename=package://unitree_ros2/description/g1/meshes/right_palm_for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
- link right_ring_1: geometry collision mesh filename=package://unitree_ros2/description/g1/meshes/right_ring_1.S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; visual mesh filename=package://unitree_ros2/description/g1/meshes/right_ring_1.S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
- link right_ring_2: geometry collision mesh filename=package://unitree_ros2/description/g1/meshes/right_ring_2.S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; visual mesh filename=package://unitree_ros2/description/g1/meshes/right_ring_2.S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
- link right_ring_force_sensor_1: geometry collision mesh filename=package://unitree_ros2/description/g1/meshes/right_ring_for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; visual mesh filename=package://unitree_ros2/description/g1/meshes/right_ring_for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
- link right_ring_force_sensor_2: geometry collision mesh filename=package://unitree_ros2/description/g1/meshes/right_ring_for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; visual mesh filename=package://unitree_ros2/description/g1/meshes/right_ring_for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
- link right_ring_force_sensor_3: geometry collision mesh filename=package://unitree_ros2/description/g1/meshes/right_ring_for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; visual mesh filename=package://unitree_ros2/description/g1/meshes/right_ring_for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
- link right_shoulder_pitch_link: geometry collision cylinder length=0.05 radius=0.03; visual mesh filename=package://unitree_ros2/description/g1/meshes/right_shoulder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
- link right_shoulder_roll_link: geometry collision cylinder length=0.03 radius=0.03; visual mesh filename=package://unitree_ros2/description/g1/meshes/right_shoulder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
- link right_shoulder_yaw_link: geometry collision mesh filename=package://unitree_ros2/description/g1/meshes/right_shoulder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; visual mesh filename=package://unitree_ros2/description/g1/meshes/right_shoulder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
- link right_thumb_1: geometry collision mesh filename=package://unitree_ros2/description/g1/meshes/right_thumb_1.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; visual mesh filename=package://unitree_ros2/description/g1/meshes/right_thumb_1.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
- link right_thumb_2: geometry collision mesh filename=package://unitree_ros2/description/g1/meshes/right_thumb_2.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; visual mesh filename=package://unitree_ros2/description/g1/meshes/right_thumb_2.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
- link right_thumb_3: geometry collision mesh filename=package://unitree_ros2/description/g1/meshes/right_thumb_3.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; visual mesh filename=package://unitree_ros2/description/g1/meshes/right_thumb_3.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
- link right_thumb_4: geometry collision mesh filename=package://unitree_ros2/description/g1/meshes/right_thumb_4.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; visual mesh filename=package://unitree_ros2/description/g1/meshes/right_thumb_4.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
- link right_thumb_force_sensor_1: geometry collision mesh filename=package://unitree_ros2/description/g1/meshes/right_thumb_fo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; visual mesh filename=package://unitree_ros2/description/g1/meshes/right_thumb_fo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
- link right_thumb_force_sensor_2: geometry collision mesh filename=package://unitree_ros2/description/g1/meshes/right_thumb_fo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; visual mesh filename=package://unitree_ros2/description/g1/meshes/right_thumb_fo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
- link right_thumb_force_sensor_3: geometry collision mesh filename=package://unitree_ros2/description/g1/meshes/right_thumb_fo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; visual mesh filename=package://unitree_ros2/description/g1/meshes/right_thumb_fo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
- link right_thumb_force_sensor_4: geometry collision mesh filename=package://unitree_ros2/description/g1/meshes/right_thumb_fo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; visual mesh filename=package://unitree_ros2/description/g1/meshes/right_thumb_fo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
- link right_wrist_pitch_link: geometry collision mesh filename=package://unitree_ros2/description/g1/meshes/right_wrist_pi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; visual mesh filename=package://unitree_ros2/description/g1/meshes/right_wrist_pi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
- link right_wrist_roll_link: geometry collision mesh filename=package://unitree_ros2/description/g1/meshes/right_wrist_ro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; visual mesh filename=package://unitree_ros2/description/g1/meshes/right_wrist_ro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
- link right_wrist_yaw_link: geometry collision mesh filename=package://unitree_ros2/description/g1/meshes/right_wrist_ya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; visual mesh filename=package://unitree_ros2/description/g1/meshes/right_wrist_ya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
- link torso_link: geometry collision mesh filename=package://unitree_ros2/description/g1/meshes/torso_link_rev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; visual mesh filename=package://unitree_ros2/description/g1/meshes/torso_link_rev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
- link waist_roll_link: geometry visual mesh filename=package://unitree_ros2/description/g1/meshes/waist_roll_lin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
- link waist_yaw_link: geometry visual mesh filename=package://unitree_ros2/description/g1/meshes/waist_yaw_link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

Commit message: added d435_cam_link

File: robots/g1_description/g1_29dof_rev_1_0_with_inspire_hand_FTP.urdf (robot description, URDF)
Before this commit: robot g1_29dof_rev_1_0_with_inspire_hand_FTP, 97 links, 96 joints
Links:
- added link d435_cam_link
Joints:
- added joint d435_cam_joint: type fixed, parent d435_link, child d435_cam_link, origin xyz=0.0 0.0 0.0 rpy=-1.570796327 0 -1.570796327

Commit message: changed Lidar frame orientation

File: robots/g1_description/g1_29dof_rev_1_0_with_inspire_hand_FTP.urdf (robot description, URDF)
Before this commit: robot g1_29dof_rev_1_0_with_inspire_hand_FTP, 98 links, 97 joints
Joints:
- joint mid360_joint: origin xyz=0.0002835 0.00003 0.41618 rpy=0 0.04014257279586953 0 -> xyz=0.0002835 0.00003 0.41618 rpy=3.1415926536 0.04014257279586953 0

Commit message: fixed inspire hand joint speeds

File: robots/g1_description/g1_29dof_rev_1_0_with_inspire_hand_FTP.urdf (robot description, URDF)
Before this commit: robot g1_29dof_rev_1_0_with_inspire_hand_FTP, 98 links, 97 joints
Joints:
- joint left_index_1_joint: limit lower=0 upper=1.4381 effort=10 velocity=1 -> lower=0 upper=1.4381 effort=10 velocity=10
- joint left_index_2_joint: limit lower=0 upper=3.14 effort=10 velocity=1 -> lower=0 upper=3.14 effort=10 velocity=10
- joint left_little_1_joint: limit lower=0 upper=1.4381 effort=10 velocity=1 -> lower=0 upper=1.4381 effort=10 velocity=10
- joint left_little_2_joint: limit lower=0 upper=3.14 effort=10 velocity=1 -> lower=0 upper=3.14 effort=10 velocity=10
- joint left_middle_1_joint: limit lower=0 upper=1.4381 effort=10 velocity=1 -> lower=0 upper=1.4381 effort=10 velocity=10
- joint left_middle_2_joint: limit lower=0 upper=3.14 effort=10 velocity=1 -> lower=0 upper=3.14 effort=10 velocity=10
- joint left_ring_1_joint: limit lower=0 upper=1.4381 effort=10 velocity=1 -> lower=0 upper=1.4381 effort=10 velocity=10
- joint left_ring_2_joint: limit lower=0 upper=3.14 effort=10 velocity=1 -> lower=0 upper=3.14 effort=10 velocity=10
- joint left_thumb_1_joint: limit lower=0 upper=1.1641 effort=10 velocity=1 -> lower=0 upper=1.1641 effort=10 velocity=10
- joint left_thumb_2_joint: limit lower=0 upper=0.5864 effort=10 velocity=1 -> lower=0 upper=0.5864 effort=10 velocity=10
- joint left_thumb_3_joint: limit lower=0 upper=0.5 effort=10 velocity=1 -> lower=0 upper=0.5 effort=10 velocity=10
- joint left_thumb_4_joint: limit lower=0 upper=3.14 effort=10 velocity=1 -> lower=0 upper=3.14 effort=10 velocity=10
- joint right_index_1_joint: limit lower=0 upper=1.4381 effort=10 velocity=1 -> lower=0 upper=1.4381 effort=10 velocity=10
- joint right_index_2_joint: limit lower=0 upper=3.14 effort=10 velocity=1 -> lower=0 upper=3.14 effort=10 velocity=10
- joint right_little_1_joint: limit lower=0 upper=1.4381 effort=10 velocity=1 -> lower=0 upper=1.4381 effort=10 velocity=10
- joint right_little_2_joint: limit lower=0 upper=3.14 effort=10 velocity=1 -> lower=0 upper=3.14 effort=10 velocity=10
- joint right_middle_1_joint: limit lower=0 upper=1.4381 effort=10 velocity=1 -> lower=0 upper=1.4381 effort=10 velocity=10
- joint right_middle_2_joint: limit lower=0 upper=3.14 effort=10 velocity=1 -> lower=0 upper=3.14 effort=10 velocity=10
- joint right_ring_1_joint: limit lower=0 upper=1.4381 effort=10 velocity=1 -> lower=0 upper=1.4381 effort=10 velocity=10
- joint right_ring_2_joint: limit lower=0 upper=3.14 effort=10 velocity=1 -> lower=0 upper=3.14 effort=10 velocity=10
- joint right_thumb_1_joint: limit lower=0 upper=1.1641 effort=10 velocity=1 -> lower=0 upper=1.1641 effort=10 velocity=10
- joint right_thumb_2_joint: limit lower=0 upper=0.5864 effort=10 velocity=1 -> lower=0 upper=0.5864 effort=10 velocity=10
- joint right_thumb_3_joint: limit lower=0 upper=0.5 effort=10 velocity=1 -> lower=0 upper=0.5 effort=10 velocity=10
- joint right_thumb_4_joint: limit lower=0 upper=3.14 effort=10 velocity=1 -> lower=0 upper=3.14 effort=10 velocity=10
